File: RGBW Driver.kicad_pcb (KiCad board)
At the start: 2 copper layers, 22.1 x 59.5 mm, 25 parts, among them J1 LED, J2 LED, J3 LED, J4 LED, J5 Power, U1 PT4115, U2 PT4115, U3 PT4115, U4 PT4115

Commit message: single and double versions
Routing:
- net /Vin: track 172.2 -> 126.0 mm
- net /Gnd: track 143.9 -> 145.0 mm, vias 40 -> 44
Other:
- board text added: "+"
- board text added: "-"
- board text added: "1"
- board text added: "2"
- board text added: "3"
- board text added: "4"
- board text added: "Eagle Decorations RGBW 1 AMP LED Driver V1.0"
